File: pcb/power-supply.kicad_sch (KiCad schematic)
At the start: 7 parts, among them CN24 KF2EDGV-3.5-2P, U11 LM2596S-5

Commit message: Fix part number.
Parts:
- C2: LCSC Part C340768 -> C8028
Changed lines of the file:
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@@
       (effects (font (size 1.27 1.27)) (justify left))
     )
-    (property "LCSC Part" "C340768" (at 144.145 46.355 0)
+    (property "LCSC Part" "C8028" (at 144.145 46.355 0)
       (effects (font (size 1.27 1.27)) hide)
     )
