File: pcb/door-adapter/door-adapter.kicad_pcb (KiCad board)
At the start: 2 copper layers, 26 x 72 mm, 10 parts, among them CN1 KF2EDGV-3.5-2P, CN2 KF2EDGV-3.5-4P, CN3 KF2EDGV-3.5-2P, CN4 KF2EDGV-3.5-2P, CN5 KF2EDGA-3.5-2P, CN6 KF2EDGR-3.5-2P, Q1 PMOS, U1 PC817C

Commit message: Add order number placeholder.
Other:
- board text added: "JLCJLCJLCJLC"
Changed lines of the file:
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@@
   (gr_arc (start 114 100) (mid 115.414214 100.585786) (end 116 102)
     (stroke (width 0.1) (type default)) (layer "Edge.Cuts"))
+  (gr_text "JLCJLCJLCJLC" (at 103 170) (layer "B.SilkS")
+    (effects (font (size 1 1) (thickness 0.15)) (justify bottom))
+  )
   (gr_text "VCC" (at 112.25 110 90) (layer "F.SilkS")
     (effects (font (face "Alte Haas Grotesk") (size 1 1) (thickness 0.15)) (justify right))
